Commit message: Basic setup for pick and place complete

File: arm_urdf/urdf/ArmPlate.xacro (robot description, xacro)
@@ -172,4 +172,16 @@
         </collision>
     </link>
+    <link name="grasp_frame">
+        <visual name="sphere">
+            <geometry>
+                <sphere radius="0.01"/>
+            </geometry>
+        </visual>
+    </link>
+    <joint name="grasp_joint" type="fixed">
+        <origin xyz="0.0 0.0 0.125" rpy="0.0 0.0 0.0" />
+        <parent link="gripperHousing-v2" />
+        <child link="grasp_frame" />
+    </joint>
     <joint name="Base_link1-v1_Revolute-1" type="continuous">
         <origin xyz="-0.05188764 -0.052144760000000005 0.01" rpy="3.141592653589793 -0.0 0.0" />

Commit message: Fixed prismatic joint issue

File: arm_urdf/urdf/ArmPlate.xacro (robot description, xacro)
@@ -1,4 +1,9 @@
 <?xml version='1.0' encoding='utf-8'?>
 <robot name="ArmPlate">
+    <link name="world"/>
+    <joint name="base_to_world" type="fixed">
+        <parent link="world" />
+        <child link="Base_link1-v1" />
+    </joint>
     <link name="Base_link1-v1">
         <inertial>
@@ -225,5 +230,5 @@
         <child link="left_H-v1" />
         <axis xyz="1.0132025937202353e-16 0.077572 0.996987" />
-        <limit lower="-0.11" upper="-0.07" effort="1000000" velocity="1000000" />
+        <limit upper="0.07" lower="-0.04" effort="10" velocity="10" />
     </joint>
     <joint name="gripperHousing-v2_Slider-14" type="prismatic">
@@ -232,5 +237,6 @@
         <child link="right_H-v1" />
         <axis xyz="2.0264051874404916e-16 -0.077572 0.996987" />
-        <limit lower="-0.11" upper="-0.07" effort="1000000" velocity="1000000" />
+        <limit upper="0.07" lower="-0.04" effort="10" velocity="10" />
+        <mimic joint="gripperHousing-v2_Slider-13" />
     </joint>
 </robot>

File: arm_urdf_moveit_config/config/ArmPlate.ros2_control.xacro (robot description, xacro)
@@ -57,11 +57,4 @@
                 <state_interface name="velocity"/>
             </joint>
-            <joint name="gripperHousing-v2_Slider-14">
-                <command_interface name="position"/>
-                <state_interface name="position">
-                  <param name="initial_value">${initial_positions['gripperHousing-v2_Slider-14']}</param>
-                </state_interface>
-                <state_interface name="velocity"/>
-            </joint>
         </ros2_control>
     </xacro:macro>

Commit message: Pick and Place completed

File: arm_urdf/urdf/ArmPlate.xacro (robot description, xacro)
@@ -178,12 +178,7 @@
     </link>
     <link name="grasp_frame">
-        <visual name="sphere">
-            <geometry>
-                <sphere radius="0.01"/>
-            </geometry>
-        </visual>
     </link>
     <joint name="grasp_joint" type="fixed">
-        <origin xyz="0.0 0.0 0.125" rpy="0.0 0.0 0.0" />
+        <origin xyz="0.0 0.0 0.15" rpy="0.0 0.0 0.0" />
         <parent link="gripperHousing-v2" />
         <child link="grasp_frame" />
